File: FroggyRun/MainBoard.brd (EAGLE design)
At the start: 73.7 x 61 mm, 18 parts

Commit message: ghkj
Parts:
- removed CAPACITOR: 1X2, FroggyRun:1X02_LONGPADS
- added C1: (no value), rcl:C025-024X044
- renumbered U$8 to USBPOWER
Connections:
- net N$15 renamed RESET
- net N$16 renamed RX
- net N$17 renamed TX
- removed net N$20: CAPACITOR.1, U$1.8, USBPOWER.GND
- removed net N$21: CAPACITOR.2, U$1.7, USBPOWER.5V
- new net USBPOWER: USBPOWER.5V
- net GND: now also C1.2, U$1.8, USBPOWER.GND
- net VIN: now also C1.1, U$1.7
Routing:
- net N$20: track 39.6 -> 0.00 mm
- net N$21: track 36.9 -> 0.00 mm
- net RESET: track 12.9 -> 11.8 mm
- net VIN: track 109.0 -> 108.0 mm
Changed lines of the file:
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@@
 <attribute name="VALUE" x="17.653" y="39.497" size="0.6096" layer="27" font="vector" ratio="20" rot="R270"/>
-</element>
-<element name="CAPACITOR" library="FroggyRun" package="1X02_LONGPADS" value="1X2" x="45.72" y="34.29" smashed="yes" rot="R270">
-<attribute name="NAME" x="47.752" y="35.56" size="0.6096" layer="25" font="vector" ratio="20" rot="R270"/>
-<attribute name="VALUE" x="43.053" y="35.687" size="0.6096" layer="27" font="vector" ratio="20" rot="R270"/>
 </element>
 <element name="LEDSTRIP" library="FroggyRun" package="1X03_NO_SILK" value="1X3" x="13.97" y="41.91" smashed="yes" rot="R270">
@@
 </element>
 <element name="U$7" library="FroggyRun" package="BUTTON" value="BUTTON" x="36.83" y="3.81" smashed="yes" rot="R90"/>
-<element name="U$8" library="FroggyRun" package="USB" value="USB" x="73.66" y="41.91" smashed="yes" rot="R270"/>
+<element name="USBPOWER" library="FroggyRun" package="USB" value="USB" x="73.66" y="41.91" smashed="yes" rot="R270"/>
+<element name="C1" library="rcl" library_urn="urn:adsk.eagle:library:334" package="C025-024X044" package3d_urn="urn:adsk.eagle:package:23630/1" value="" x="3.81" y="-17.78" smashed="yes">
+<attribute name="NAME" x="2.032" y="-16.383" size="1.27" layer="25" ratio="10"/>
+<attribute name="SPICEPREFIX" value="C" x="3.81" y="-17.78" size="1.778" layer="27" display="off"/>
+<attribute name="VALUE" x="2.032" y="-20.447" size="1.27" layer="27" ratio="10"/>
+</element>
 </elements>
 <signals>
@@
 <wire x1="15.0045" y1="25.722" x2="15.0045" y2="20.006" width="0.635" layer="16"/>
 <wire x1="36.4395" y1="4.287" x2="36.83" y2="3.81" width="0.635" layer="16"/>
+<contactref element="C1" pad="2"/>
+<contactref element="U$1" pad="8"/>
+<contactref element="USBPOWER" pad="GND"/>
+<wire x1="48.586" y1="41.441" x2="71.12" y2="46.99" width="0" layer="19" extent="16-16"/>
+<wire x1="36.83" y1="34.29" x2="29.21" y2="31.75" width="0" layer="19" extent="1-1"/>
+<wire x1="5.08" y1="-17.78" x2="28.58" y2="6.4305" width="0" layer="19" extent="16-16"/>
 </signal>
 <signal name="N$11">
@@
 <contactref element="LEDSTRIP" pad="3"/>
 <contactref element="OLED" pad="VIN"/>
-<contactref element="U$6" pad="P$2"/>
 <contactref element="PROGRAMMING" pad="4"/>
 <wire x1="43.5845" y1="7.8595" x2="42.1555" y2="7.8595" width="0.635" layer="16"/>
 <wire x1="47.157" y1="11.432" x2="43.5845" y2="7.8595" width="0.635" layer="16"/>
 <wire x1="47.8715" y1="11.432" x2="47.157" y2="11.432" width="0.635" layer="16"/>
-<wire x1="42.1555" y1="7.8595" x2="41.91" y2="7.62" width="0.635" layer="16"/>
 <wire x1="47.8715" y1="11.432" x2="48.26" y2="11.43" width="0.635" layer="16"/>
 <wire x1="13.5755" y1="34.296" x2="13.5755" y2="36.4395" width="0.635" layer="16"/>
@@
 <wire x1="32.1525" y1="35.725" x2="32.1525" y2="10.003" width="0.635" layer="16"/>
 <wire x1="30.7235" y1="37.154" x2="32.1525" y2="35.725" width="0.635" layer="16"/>
-<wire x1="41.441" y1="7.145" x2="41.91" y2="7.62" width="0.635" layer="16"/>
+<contactref element="U$6" pad="P$2"/>
+<contactref element="C1" pad="1"/>
+<contactref element="U$1" pad="7"/>
+<wire x1="32.1525" y1="35.725" x2="36.83" y2="31.75" width="0" layer="19" extent="16-16"/>
+<wire x1="41.91" y1="7.62" x2="41.441" y2="7.145" width="0" layer="19" extent="16-16"/>
+<wire x1="42.1555" y1="7.8595" x2="41.91" y2="7.62" width="0" layer="19" extent="16-16"/>
+<wire x1="2.54" y1="-17.78" x2="32.1525" y2="10.003" width="0" layer="19" extent="16-16"/>
 </signal>
 <signal name="N$1">
@@
 <wire x1="67.163" y1="29.2945" x2="67.31" y2="29.21" width="0.635" layer="16"/>
 </signal>
-<signal name="N$15">
+<signal name="RESET">
 <contactref element="U$1" pad="1"/>
-<contactref element="U$6" pad="P$1"/>
-<contactref element="U$7" pad="P$2"/>
 <wire x1="37.154" y1="16.4335" x2="37.154" y2="15.719" width="0.635" layer="16"/>
 <wire x1="37.154" y1="15.719" x2="37.154" y2="9.2885" width="0.635" layer="16"/>
-<wire x1="37.154" y1="9.2885" x2="36.83" y2="8.89" width="0.635" layer="16"/>
 <wire x1="37.154" y1="16.4335" x2="36.83" y2="16.51" width="0.635" layer="16"/>
 <wire x1="37.154" y1="15.719" x2="41.441" y2="15.719" width="0.635" layer="16"/>
-<wire x1="41.441" y1="15.719" x2="41.91" y2="15.24" width="0.635" layer="16"/>
-</signal>
-<signal name="N$16">
+<contactref element="U$7" pad="P$2"/>
+<contactref element="U$6" pad="P$1"/>
+<wire x1="41.441" y1="15.719" x2="41.91" y2="15.24" width="0" layer="19" extent="16-16"/>
+<wire x1="36.83" y1="8.89" x2="37.154" y2="9.2885" width="0" layer="19" extent="16-16"/>
+</signal>
+<signal name="RX">
 <contactref element="U$1" pad="2"/>
 <contactref element="PROGRAMMING" pad="3"/>
@@
 <wire x1="37.154" y1="18.577" x2="36.83" y2="19.05" width="0.635" layer="16"/>
 </signal>
-<signal name="N$17">
+<signal name="TX">
 <contactref element="U$1" pad="3"/>
 <contactref element="PROGRAMMING" pad="2"/>
@@
 <wire x1="45.0135" y1="42.1555" x2="45.72" y2="41.91" width="0.635" layer="16"/>
 </signal>
-<signal name="N$21">
-<contactref element="U$1" pad="7"/>
-<contactref element="CAPACITOR" pad="2"/>
-<contactref element="U$8" pad="5V"/>
-<wire x1="45.0135" y1="32.1525" x2="37.154" y2="32.1525" width="0.635" layer="16"/>
-<wire x1="37.154" y1="32.1525" x2="36.83" y2="31.75" width="0.635" layer="16"/>
-<wire x1="45.0135" y1="32.1525" x2="45.72" y2="31.75" width="0.635" layer="16"/>
-<wire x1="51.444" y1="36.4395" x2="70.7355" y2="36.4395" width="0.635" layer="16"/>
-<wire x1="47.157" y1="32.1525" x2="51.444" y2="36.4395" width="0.635" layer="16"/>
-<wire x1="45.728" y1="32.1525" x2="47.157" y2="32.1525" width="0.635" layer="16"/>
-<wire x1="70.7355" y1="36.4395" x2="71.12" y2="36.83" width="0.635" layer="16"/>
-<wire x1="45.728" y1="32.1525" x2="45.72" y2="31.75" width="0.635" layer="16"/>
-</signal>
-<signal name="N$20">
-<contactref element="U$1" pad="8"/>
-<contactref element="CAPACITOR" pad="1"/>
-<contactref element="U$8" pad="GND"/>
-<wire x1="45.0135" y1="34.296" x2="37.154" y2="34.296" width="0.635" layer="16"/>
-<wire x1="37.154" y1="34.296" x2="36.83" y2="34.29" width="0.635" layer="16"/>
-<wire x1="45.0135" y1="34.296" x2="45.72" y2="34.29" width="0.635" layer="16"/>
-<wire x1="58.589" y1="46.4425" x2="70.7355" y2="46.4425" width="0.635" layer="16"/>
-<wire x1="46.4425" y1="34.296" x2="58.589" y2="46.4425" width="0.635" layer="16"/>
-<wire x1="45.728" y1="34.296" x2="46.4425" y2="34.296" width="0.635" layer="16"/>
-<wire x1="70.7355" y1="46.4425" x2="71.12" y2="46.99" width="0.635" layer="16"/>
-<wire x1="45.728" y1="34.296" x2="45.72" y2="34.29" width="0.635" layer="16"/>
+<signal name="USBPOWER">
+<contactref element="USBPOWER" pad="5V"/>
 </signal>
 </signals>
@@
 </drawing>
 <compatibility>
+<note version="8.2" severity="warning">
+Since Version 8.2, EAGLE supports online libraries. The ids
+of those online libraries will not be understood (or retained)
+with this version.
+</note>
 <note version="8.3" severity="warning">
 Since Version 8.3, EAGLE supports URNs for individual library
@@
 will not be understood (or retained) with this version.
 </note>
+<note version="8.3" severity="warning">
+Since Version 8.3, EAGLE supports the association of 3D packages
+with devices in libraries, schematics, and board files. Those 3D
+packages will not be understood (or retained) with this version.
+</note>
 </compatibility>
