File: FroggyRun/Boardv2.sch (EAGLE design)
At the start: 18 parts

Commit message: gkl,fdfalkj;
Parts:
- renumbered RESET to U$3
Connections:
- net 5V: now also RESISTOR.2; no longer U$3.1
- net GND: now also U$3.1; no longer RESISTOR.2
Changed lines of the file:
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@@
 <parts>
 <part name="U$1" library="FroggyRun" deviceset="ATMEGA328" device=""/>
-<part name="RESET" library="FroggyRun" deviceset="MOMENTARY_SWITCH" device=""/>
 <part name="RESISTOR" library="FroggyRun" deviceset="RESISTOR" device="" value="10k"/>
 <part name="SUPPLY1" library="SparkFun-PowerSymbols" library_urn="urn:adsk.eagle:library:530" deviceset="5V" device=""/>
@@
 <part name="SUPPLY9" library="SparkFun-PowerSymbols" library_urn="urn:adsk.eagle:library:530" deviceset="5V" device=""/>
 <part name="GND14" library="SparkFun-PowerSymbols" library_urn="urn:adsk.eagle:library:530" deviceset="GND" device=""/>
+<part name="U$3" library="FroggyRun" deviceset="MOMENTARY_SWITCH" device=""/>
 </parts>
 <sheets>
@@
 <instances>
 <instance part="U$1" gate="G$1" x="38.1" y="22.86" smashed="yes"/>
-<instance part="RESET" gate="G$2" x="53.34" y="12.7" smashed="yes">
-<attribute name="NAME" x="53.34" y="14.224" size="1.778" layer="95" font="vector" align="bottom-center"/>
-<attribute name="VALUE" x="53.34" y="12.192" size="1.778" layer="96" font="vector" align="top-center"/>
-</instance>
 <instance part="RESISTOR" gate="G$1" x="71.12" y="5.08" smashed="yes" rot="R270">
 <attribute name="NAME" x="72.644" y="5.08" size="1.778" layer="95" font="vector" rot="R270" align="bottom-center"/>
 <attribute name="VALUE" x="69.596" y="5.08" size="1.778" layer="96" font="vector" rot="R270" align="top-center"/>
 </instance>
-<instance part="SUPPLY1" gate="G$1" x="43.18" y="15.24" smashed="yes">
-<attribute name="VALUE" x="43.18" y="18.034" size="1.778" layer="96" align="bottom-center"/>
-</instance>
-<instance part="GND2" gate="1" x="71.12" y="-5.08" smashed="yes">
-<attribute name="VALUE" x="71.12" y="-5.334" size="1.778" layer="96" align="top-center"/>
+<instance part="SUPPLY1" gate="G$1" x="63.5" y="0" smashed="yes">
+<attribute name="VALUE" x="63.5" y="2.794" size="1.778" layer="96" align="bottom-center"/>
+</instance>
+<instance part="GND2" gate="1" x="40.64" y="7.62" smashed="yes">
+<attribute name="VALUE" x="40.64" y="7.366" size="1.778" layer="96" align="top-center"/>
 </instance>
 <instance part="PROGRAMMING" gate="G$1" x="88.9" y="22.86" smashed="yes" rot="R180">
@@
 <instance part="GND14" gate="1" x="10.16" y="38.1" smashed="yes">
 <attribute name="VALUE" x="10.16" y="37.846" size="1.778" layer="96" align="top-center"/>
+</instance>
+<instance part="U$3" gate="G$2" x="53.34" y="12.7" smashed="yes">
+<attribute name="NAME" x="53.34" y="14.224" size="1.778" layer="95" font="vector" align="bottom-center"/>
+<attribute name="VALUE" x="53.34" y="12.192" size="1.778" layer="96" font="vector" align="top-center"/>
 </instance>
 </instances>
@@
 <pinref part="RESISTOR" gate="G$1" pin="1"/>
 <wire x1="71.12" y1="22.86" x2="71.12" y2="12.7" width="0.1524" layer="91"/>
-<pinref part="RESET" gate="G$2" pin="2"/>
 <wire x1="71.12" y1="12.7" x2="71.12" y2="10.16" width="0.1524" layer="91"/>
 <wire x1="58.42" y1="12.7" x2="71.12" y2="12.7" width="0.1524" layer="91"/>
 <junction x="71.12" y="12.7"/>
 <label x="66.04" y="22.86" size="1.778" layer="95"/>
+<pinref part="U$3" gate="G$2" pin="2"/>
 </segment>
 </net>
 <net name="5V" class="0">
-<segment>
-<pinref part="RESET" gate="G$2" pin="1"/>
-<wire x1="48.26" y1="12.7" x2="43.18" y2="12.7" width="0.1524" layer="91"/>
-<pinref part="SUPPLY1" gate="G$1" pin="5V"/>
-<wire x1="43.18" y1="12.7" x2="43.18" y2="15.24" width="0.1524" layer="91"/>
-</segment>
 <segment>
 <pinref part="SUPPLY2" gate="G$1" pin="5V"/>
@@
 <pinref part="SUPPLY9" gate="G$1" pin="5V"/>
 </segment>
+<segment>
+<pinref part="SUPPLY1" gate="G$1" pin="5V"/>
+<wire x1="63.5" y1="0" x2="63.5" y2="-2.54" width="0.1524" layer="91"/>
+<wire x1="63.5" y1="-2.54" x2="71.12" y2="-2.54" width="0.1524" layer="91"/>
+<pinref part="RESISTOR" gate="G$1" pin="2"/>
+<wire x1="71.12" y1="-2.54" x2="71.12" y2="0" width="0.1524" layer="91"/>
+</segment>
 </net>
 <net name="GND" class="0">
-<segment>
-<pinref part="RESISTOR" gate="G$1" pin="2"/>
-<pinref part="GND2" gate="1" pin="GND"/>
-<wire x1="71.12" y1="0" x2="71.12" y2="-2.54" width="0.1524" layer="91"/>
-</segment>
 <segment>
 <pinref part="PROGRAMMING" gate="G$1" pin="6"/>
@@
 <pinref part="GND14" gate="1" pin="GND"/>
 </segment>
+<segment>
+<wire x1="48.26" y1="12.7" x2="40.64" y2="12.7" width="0.1524" layer="91"/>
+<pinref part="GND2" gate="1" pin="GND"/>
+<wire x1="40.64" y1="12.7" x2="40.64" y2="10.16" width="0.1524" layer="91"/>
+<pinref part="U$3" gate="G$2" pin="1"/>
+</segment>
 </net>
